File: dev-board/pcb/25.sch (KiCad schematic (older format))
At the start: 2 parts, among them U5 25LCxxx

Commit message: Replace RN1 with 4 0804 resistors
Closes #9
Changed lines of the file:
@@
 AR Path="/5D73BD77/5E08F69E" Ref="U14"  Part="1"
 AR Path="/5D73BD8B/5E08F69E" Ref="U13"  Part="1"
-F 0 "U5" H 4900 4200 50  0000 C CNN
+F 0 "U20" H 4900 4200 50  0000 C CNN
 F 1 "25LCxxx" H 5350 4200 50  0000 C CNN
 F 2 "Package_SO:SOIC-8_3.9x4.9mm_P1.27mm" H 5150 3950 50  0001 C CNN
@@
 AR Path="/5D73BD77/5E0FC1AC" Ref="C17"  Part="1"
 AR Path="/5D73BD8B/5E0FC1AC" Ref="C16"  Part="1"
-F 0 "C6" H 4315 3996 50  0000 L CNN
+F 0 "C23" H 4315 3996 50  0000 L CNN
 F 1 "100n" H 4315 3905 50  0000 L CNN
 F 2 "Capacitor_SMD:C_0805_2012Metric_Pad1.15x1.40mm_HandSolder" H 4238 3800 50  0001 C CNN
